File: Outputs_analog_24V_8pcs/Outputs.sch (KiCad schematic (older format))
At the start: 112 parts, among them J10 Screw_Terminal_01x02, J11 Screw_Terminal_01x02, J4 Screw_Terminal_01x02, J5 Screw_Terminal_01x02, J6 Screw_Terminal_01x02, J7 Screw_Terminal_01x02, J8 Screw_Terminal_01x02, J9 Screw_Terminal_01x02, Q1 2SK2800, Q2 2SK2800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

Commit message: Update Outputs pcb
Parts:
- D11, D13, D15, D17, D3, D5, D7, D9: footprint Diode_THT:D_A-405_P2.54mm_Vertical_AnodeUp -> LED_THT:LED_D3.0mm
Changed lines of the file:
@@
 EESchema Schematic File Version 4
-EELAYER 30 0
+LIBS:Outputs_analog_24V_8pcs-cache
+EELAYER 26 0
 EELAYER END
 $Descr A4 8268 11693 portrait
@@
 F 0 "D3" V 1047 1678 50  0000 L CNN
 F 1 "LED" V 1138 1678 50  0000 L CNN
-F 2 "Diode_THT:D_A-405_P2.54mm_Vertical_AnodeUp" H 1100 1600 50  0001 C CNN
+F 2 "LED_THT:LED_D3.0mm" H 1100 1600 50  0001 C CNN
 F 3 "~" H 1100 1600 50  0001 C CNN
 	1    1100 1600
@@
 F 0 "D5" V 1047 3728 50  0000 L CNN
 F 1 "LED" V 1138 3728 50  0000 L CNN
-F 2 "Diode_THT:D_A-405_P2.54mm_Vertical_AnodeUp" H 1100 3650 50  0001 C CNN
+F 2 "LED_THT:LED_D3.0mm" H 1100 3650 50  0001 C CNN
 F 3 "~" H 1100 3650 50  0001 C CNN
 	1    1100 3650
@@
 F 0 "D7" V 1047 5778 50  0000 L CNN
 F 1 "LED" V 1138 5778 50  0000 L CNN
-F 2 "Diode_THT:D_A-405_P2.54mm_Vertical_AnodeUp" H 1100 5700 50  0001 C CNN
+F 2 "LED_THT:LED_D3.0mm" H 1100 5700 50  0001 C CNN
 F 3 "~" H 1100 5700 50  0001 C CNN
 	1    1100 5700
@@
 F 0 "D9" V 1047 7828 50  0000 L CNN
 F 1 "LED" V 1138 7828 50  0000 L CNN
-F 2 "Diode_THT:D_A-405_P2.54mm_Vertical_AnodeUp" H 1100 7750 50  0001 C CNN
+F 2 "LED_THT:LED_D3.0mm" H 1100 7750 50  0001 C CNN
 F 3 "~" H 1100 7750 50  0001 C CNN
 	1    1100 7750
@@
 F 0 "D11" V 4497 1678 50  0000 L CNN
 F 1 "LED" V 4588 1678 50  0000 L CNN
-F 2 "Diode_THT:D_A-405_P2.54mm_Vertical_AnodeUp" H 4550 1600 50  0001 C CNN
+F 2 "LED_THT:LED_D3.0mm" H 4550 1600 50  0001 C CNN
 F 3 "~" H 4550 1600 50  0001 C CNN
 	1    4550 1600
@@
 F 0 "D13" V 4497 3728 50  0000 L CNN
 F 1 "LED" V 4588 3728 50  0000 L CNN
-F 2 "Diode_THT:D_A-405_P2.54mm_Vertical_AnodeUp" H 4550 3650 50  0001 C CNN
+F 2 "LED_THT:LED_D3.0mm" H 4550 3650 50  0001 C CNN
 F 3 "~" H 4550 3650 50  0001 C CNN
 	1    4550 3650
@@
 F 0 "D15" V 4497 5778 50  0000 L CNN
 F 1 "LED" V 4588 5778 50  0000 L CNN
-F 2 "Diode_THT:D_A-405_P2.54mm_Vertical_AnodeUp" H 4550 5700 50  0001 C CNN
+F 2 "LED_THT:LED_D3.0mm" H 4550 5700 50  0001 C CNN
 F 3 "~" H 4550 5700 50  0001 C CNN
 	1    4550 5700
@@
 F 0 "D17" V 4497 7828 50  0000 L CNN
 F 1 "LED" V 4588 7828 50  0000 L CNN
-F 2 "Diode_THT:D_A-405_P2.54mm_Vertical_AnodeUp" H 4550 7750 50  0001 C CNN
+F 2 "LED_THT:LED_D3.0mm" H 4550 7750 50  0001 C CNN
 F 3 "~" H 4550 7750 50  0001 C CNN
 	1    4550 7750
