File: Outputs_analog_24V_8pcs/Outputs_analog_24V_8pcs.kicad_pcb (KiCad board)
At the start: 2 copper layers, 146.1 x 101.6 mm, 122 parts, among them J1 Screw_Terminal_01x02, J10 Screw_Terminal_01x02, J11 Screw_Terminal_01x02, J2 Screw_Terminal_01x02, J3 Screw_Terminal_01x06, J4 Screw_Terminal_01x02, J5 Screw_Terminal_01x02, J6 Screw_Terminal_01x02, J7 Screw_Terminal_01x02, J8 Screw_Terminal_01x02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

Commit message: Update Outputs pcb
Parts:
- D1, D11, D13, D15, D17, D2, D3, D5, D7, D9: footprint Diode_THT:D_A-405_P2.54mm_Vertical_AnodeUp -> LED_THT:LED_D3.0mm
- moved D12 354.7 mm to (160.0, 92.7)
- moved R49 328.1 mm to (152.4, 80.6)
- moved Q6 327.4 mm to (134.6, 80.6), turned to 270 degrees
- moved Q5 327.3 mm to (163.2, 80.6), turned to 270 degrees
- moved R72 321.5 mm to (177.8, 69.2), turned to 270 degrees
- moved R56 312.4 mm to (177.8, 80.0), turned to 270 degrees
- moved R63 311.5 mm to (140.3, 69.2), turned to 270 degrees
- moved R69 304.8 mm to (145.4, 69.2), turned to 270 degrees
- moved R48 302.8 mm to (171.4, 92.7), turned to 270 degrees
- moved U6 302.7 mm to (174.0, 80.0), turned to 270 degrees
- moved R44 292.9 mm to (160.0, 77.5), turned to 180 degrees
- moved R68 290.2 mm to (174.0, 69.2), turned to 270 degrees
- moved R50 289.6 mm to (142.9, 92.7), turned to 270 degrees
- moved U7 288.9 mm to (145.4, 80.0), turned to 270 degrees
- moved U9 287.6 mm to (88.3, 80.0), turned to 270 degrees
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Connections:
- U1 pad 1: Net-(U1-Pad1) -> output_5
- U1 pad 10: Net-(J3-Pad3) -> Net-(J3-Pad5)
- U1 pad 11: Net-(J3-Pad2) -> Net-(J3-Pad3)
- U1 pad 12: Net-(J3-Pad4) -> Net-(J3-Pad2)
- U1 pad 13: Net-(J3-Pad5) -> Net-(J3-Pad1)
- U1 pad 14: Net-(J3-Pad1) -> Net-(J3-Pad6)
- U1 pad 15: Net-(U1-Pad15) -> output_8
- U1 pad 2: Net-(U1-Pad2) -> output_6
- U1 pad 3: Net-(U1-Pad3) -> output_7
- U1 pad 4: Net-(U1-Pad4) -> output_4
- U1 pad 5: Net-(U1-Pad5) -> output_3
- U1 pad 6: Net-(U1-Pad6) -> output_2
- U1 pad 7: Net-(U1-Pad7) -> output_1
- U1 pad 9: Net-(J3-Pad6) -> Net-(J3-Pad4)
Routing:
- net Earth: track 182.4 -> 919.5 mm
- net GND: track 51.9 -> 407.8 mm
- net +24V: track 157.5 -> 366.4 mm
- net +5V: track 0.00 -> 32.8 mm
- net Net-(J3-Pad6): track 0.00 -> 27.2 mm
- net Net-(J3-Pad1): track 0.00 -> 24.9 mm
- net Net-(D12-Pad1): track 0.00 -> 22.8 mm
- net Net-(D16-Pad1): track 0.00 -> 22.3 mm
- net Net-(D14-Pad1): track 0.00 -> 22.2 mm
- net Net-(D18-Pad1): track 0.00 -> 22.2 mm
- net Net-(J3-Pad2): track 0.00 -> 21.6 mm
- net Net-(Q6-Pad2): track 0.00 -> 18.9 mm
- net Net-(Q7-Pad2): track 0.00 -> 18.9 mm
- net Net-(Q8-Pad2): track 0.00 -> 18.9 mm
- net Net-(Q5-Pad2): track 0.00 -> 18.9 mm
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Other:
- board size 146.1 x 101.6 mm -> 158.8 x 102.9 mm

Commit message: Update pcb
Connections:
- U1 pad 1: output_5 -> output_6
- U1 pad 15: output_8 -> output_5
- U1 pad 2: output_6 -> output_8
- U1 pad 4: output_4 -> output_2
- U1 pad 6: output_2 -> output_4
Routing:
- net output_5: track 5.54 -> 129.5 mm
- net output_6: track 7.44 -> 99.0 mm
- net output_4: track 6.17 -> 89.7 mm
- net output_7: track 6.17 -> 75.7 mm
- net output_3: track 9.95 -> 56.3 mm
- net output_8: track 14.0 -> 41.9 mm
- net output_2: track 12.8 -> 23.7 mm
Other:
- board size 158.8 x 102.9 mm -> 157.5 x 72.4 mm

Commit message: Update footprints
Parts:
- J1, J10, J11, J2, J4, J5, J6, J7, J8, J9: footprint Connector_PinHeader_2.54mm:PinHeader_1x02_P2.54mm_Horizontal -> Connector_PinHeader_2.54mm:PinHeader_1x02_P2.54mm_Vertical
- J3: footprint Connector_PinHeader_2.54mm:PinHeader_1x06_P2.54mm_Horizontal -> Connector_PinHeader_2.54mm:PinHeader_1x06_P2.54mm_Vertical
