File: Inputs_analog_24V_8pcs/Inputs_analog_24V_8pcs.sch (KiCad schematic (older format))
At the start: 14 parts, among them J1 Screw_Terminal_01x02, J2 Screw_Terminal_01x02, J3 Screw_Terminal_01x06, U1 SN74HC14N, U2 SN74HC14N, U3 74HC151N.652

Commit message: Update pcb
Connections:
- net GND: now also U1.1 (1A), U1.12 (6Y), U1.13 (6A), U1.2 (1Y), U2.1 (1A), U2.12 (6Y), U2.13 (6A), U2.2 (1Y); no longer U1.3 (2A), U1.4 (2Y), U1.5 (3A), U1.6 (3Y), U2.3 (2A), U2.4 (2Y), U2.5 (3A), U2.6 (3Y)
- net input_1: now also U1.5 (3A); no longer U1.1 (1A)
- net input_2: now also U1.3 (2A); no longer U1.13 (6A)
- net input_3: now also U2.5 (3A); no longer U1.11 (5A)
- net input_4: now also U2.3 (2A); no longer U1.9 (4A)
- net input_5: now also U2.11 (5A); no longer U2.1 (1A)
- net input_6: now also U2.9 (4A); no longer U2.13 (6A)
- net input_7: now also U1.9 (4A); no longer U2.9 (4A)
- net input_8: now also U1.11 (5A); no longer U2.11 (5A)
- net at U1.10 (5Y): now also U3.14 (I5)
- net at U1.8 (4Y): now also U3.15 (I4)
- net at U2.10 (5Y): now also U3.12 (I7)
- net at U2.8 (4Y): now also U3.13 (I6)
Changed lines of the file:
@@
 F1 "Inputs.sch" 50
 $EndSheet
-Text GLabel 1500 3900 0    50   Input ~ 0
+Text GLabel 1500 3700 0    50   Input ~ 0
 input_1
-Text GLabel 1500 3400 0    50   Input ~ 0
+Text GLabel 1500 3800 0    50   Input ~ 0
 input_2
+Text GLabel 1500 5600 0    50   Input ~ 0
+input_3
+Text GLabel 1500 5700 0    50   Input ~ 0
+input_4
+Text GLabel 1500 5400 0    50   Input ~ 0
+input_5
+Text GLabel 1500 5500 0    50   Input ~ 0
+input_6
+Text GLabel 1500 3600 0    50   Input ~ 0
+input_7
 Text GLabel 1500 3500 0    50   Input ~ 0
-input_3
-Text GLabel 1500 3600 0    50   Input ~ 0
-input_4
-Text GLabel 1500 5800 0    50   Input ~ 0
-input_5
-Text GLabel 1500 5300 0    50   Input ~ 0
-input_6
-Text GLabel 1500 5500 0    50   Input ~ 0
-input_7
-Text GLabel 1500 5400 0    50   Input ~ 0
 input_8
-$Comp
-L power:GND #PWR04
-U 1 1 5EB7A823
-P 2100 6450
-F 0 "#PWR04" H 2100 6200 50  0001 C CNN
-F 1 "GND" H 2105 6277 50  0000 C CNN
-F 2 "" H 2100 6450 50  0001 C CNN
-F 3 "" H 2100 6450 50  0001 C CNN
-	1    2100 6450
-	1    0    0    -1
-$EndComp
 $Comp
 L power:+5V #PWR09
@@
 	2900 3300 3250 3300
 $Comp
-L power:GND #PWR06
-U 1 1 5EBDD6D8
-P 2900 6450
-F 0 "#PWR06" H 2900 6200 50  0001 C CNN
-F 1 "GND" H 2905 6277 50  0000 C CNN
-F 2 "" H 2900 6450 50  0001 C CNN
-F 3 "" H 2900 6450 50  0001 C CNN
-	1    2900 6450
-	1    0    0    -1
-$EndComp
-$Comp
 L Device:C C2
 U 1 1 5EBE4E47
@@
 L power:GND #PWR03
 U 1 1 5EC164A3
-P 2100 4500
-F 0 "#PWR03" H 2100 4250 50  0001 C CNN
-F 1 "GND" H 2105 4327 50  0000 C CNN
-F 2 "" H 2100 4500 50  0001 C CNN
-F 3 "" H 2100 4500 50  0001 C CNN
-	1    2100 4500
+P 2100 4250
+F 0 "#PWR03" H 2100 4000 50  0001 C CNN
+F 1 "GND" H 2105 4077 50  0000 C CNN
+F 2 "" H 2100 4250 50  0001 C CNN
+F 3 "" H 2100 4250 50  0001 C CNN
+	1    2100 4250
 	1    0    0    -1
 $EndComp
@@
 L power:GND #PWR07
 U 1 1 5E7B992E
-P 2900 4500
-F 0 "#PWR07" H 2900 4250 50  0001 C CNN
-F 1 "GND" H 2905 4327 50  0000 C CNN
-F 2 "" H 2900 4500 50  0001 C CNN
-F 3 "" H 2900 4500 50  0001 C CNN
-	1    2900 4500
+P 2900 4250
+F 0 "#PWR07" H 2900 4000 50  0001 C CNN
+F 1 "GND" H 2905 4077 50  0000 C CNN
+F 2 "" H 2900 4250 50  0001 C CNN
+F 3 "" H 2900 4250 50  0001 C CNN
+	1    2900 4250
 	1    0    0    -1
 $EndComp
@@
 $EndComp
 Connection ~ 2900 5200
-Wire Notes Line
-	5250 600  5250 1100
-Text Notes 4550 1050 0    50   ~ 0
-Optional
-Wire Notes Line
-	5250 1100 4500 1100
-Wire Notes Line
-	4500 600  4500 1100
-Wire Notes Line
-	4500 600  5250 600
 Wire Wire Line
 	2850 4000 2900 4000
-Wire Wire Line
-	2900 4000 2900 4500
-Wire Wire Line
-	2900 6450 2900 5900
 Wire Wire Line
 	2900 5900 2850 5900
@@
 	4750 3900 4750 4300
 Wire Wire Line
-	1500 3900 2150 3900
-Wire Wire Line
-	1500 3400 2150 3400
+	4700 3300 4950 3300
+Wire Wire Line
+	4700 3400 4950 3400
+Wire Wire Line
+	4700 3500 4950 3500
+Wire Wire Line
+	4700 3600 4950 3600
+Wire Wire Line
+	4700 3800 4950 3800
+Wire Wire Line
+	4700 3700 4950 3700
+Wire Wire Line
+	1500 3700 2150 3700
+Wire Wire Line
+	1500 3800 2150 3800
+Wire Wire Line
+	1500 3600 2150 3600
 Wire Wire Line
 	1500 3500 2150 3500
 Wire Wire Line
-	1500 3600 2150 3600
-Wire Wire Line
-	2100 4500 2100 3800
-Wire Wire Line
-	2100 3700 2150 3700
-Wire Wire Line
-	2150 3800 2100 3800
-Connection ~ 2100 3800
-Wire Wire Line
-	2100 3800 2100 3700
-Wire Wire Line
-	2850 3800 2900 3800
-Wire Wire Line
-	2900 3800 2900 4000
+	2150 3400 2100 3400
+Wire Wire Line
+	2100 3400 2100 3900
+Wire Wire Line
+	2150 3900 2100 3900
+Wire Wire Line
+	1500 5600 2150 5600
+Wire Wire Line
+	1500 5700 2150 5700
+Wire Wire Line
+	1500 5500 2150 5500
+Wire Wire Line
+	1500 5400 2150 5400
+Wire Wire Line
+	2150 5800 2100 5800
+Wire Wire Line
+	2150 5300 2100 5300
+Wire Wire Line
+	2100 5300 2100 5800
+Wire Wire Line
+	2850 3400 2900 3400
+Wire Wire Line
+	2900 3400 2900 3900
+Wire Wire Line
+	2850 3900 2900 3900
+Connection ~ 2900 3900
+Wire Wire Line
+	2900 3900 2900 4000
+Wire Wire Line
+	2850 5800 2900 5800
+Wire Wire Line
+	2900 5800 2900 5900
+Wire Wire Line
+	2850 5300 2900 5300
+Wire Wire Line
+	2900 5300 2900 5800
+Connection ~ 2900 5800
+Wire Wire Line
+	2850 3600 3650 3600
+Wire Wire Line
+	3650 3600 3650 3500
+Wire Wire Line
+	3650 3500 4000 3500
+Wire Wire Line
+	2850 3500 3550 3500
+Wire Wire Line
+	3550 3500 3550 3400
+Wire Wire Line
+	3550 3400 4000 3400
+Wire Wire Line
+	2850 5500 3850 5500
+Wire Wire Line
+	3850 5500 3850 3300
+Wire Wire Line
+	3850 3300 4000 3300
+Wire Wire Line
+	2850 5400 3750 5400
+Wire Wire Line
+	3750 5400 3750 3200
+Wire Wire Line
+	3750 3200 4000 3200
+Wire Notes Line
+	5600 2650 5600 3150
+Text Notes 5250 2750 0    50   ~ 0
+Optional
+Wire Notes Line
+	5600 3150 4850 3150
+Wire Notes Line
+	4850 2650 4850 3150
+Wire Notes Line
+	4850 2650 5600 2650
+Wire Notes Line
+	3700 2750 3700 3250
+Text Notes 3350 2850 0    50   ~ 0
+Optional
+Wire Notes Line
+	3700 3250 2950 3250
+Wire Notes Line
+	2950 2750 2950 3250
+Wire Notes Line
+	2950 2750 3700 2750
+Wire Wire Line
+	2100 3900 2100 4250
+Connection ~ 2100 3900
+Wire Wire Line
+	2900 4000 2900 4250
 Connection ~ 2900 4000
-Wire Wire Line
-	2850 3700 2900 3700
-Wire Wire Line
-	2900 3700 2900 3800
-Connection ~ 2900 3800
-Wire Wire Line
-	1500 5300 2150 5300
-Wire Wire Line
-	1500 5400 2150 5400
-Wire Wire Line
-	1500 5500 2150 5500
-Wire Wire Line
-	1500 5800 2150 5800
-Wire Wire Line
-	2150 5600 2100 5600
-Wire Wire Line
-	2100 5600 2100 5700
-Wire Wire Line
-	2150 5700 2100 5700
-Connection ~ 2100 5700
-Wire Wire Line
-	2100 5700 2100 6450
-Wire Wire Line
-	2850 5700 2900 5700
-Wire Wire Line
-	2900 5700 2900 5900
-Connection ~ 2900 5900
-Wire Wire Line
-	2850 5600 2900 5600
-Wire Wire Line
-	2900 5600 2900 5700
-Connection ~ 2900 5700
-Wire Wire Line
-	4700 3300 4950 3300
-Wire Wire Line
-	4700 3400 4950 3400
-Wire Wire Line
-	4700 3500 4950 3500
-Wire Wire Line
-	4700 3600 4950 3600
-Wire Wire Line
-	4700 3700 4950 3700
-Wire Wire Line
-	4700 3800 4950 3800
+Wire Notes Line
+	3700 4650 3700 5150
+Text Notes 3350 4750 0    50   ~ 0
+Optional
+Wire Notes Line
+	3700 5150 2950 5150
+Wire Notes Line
+	2950 4650 2950 5150
+Wire Notes Line
+	2950 4650 3700 4650
+$Comp
+L power:GND #PWR?
+U 1 1 5EC44226
+P 2900 6150
+F 0 "#PWR?" H 2900 5900 50  0001 C CNN
+F 1 "GND" H 2905 5977 50  0000 C CNN
+F 2 "" H 2900 6150 50  0001 C CNN
+F 3 "" H 2900 6150 50  0001 C CNN
+	1    2900 6150
+	1    0    0    -1
+$EndComp
+Wire Wire Line
+	2900 5900 2900 6150
+$Comp
+L power:GND #PWR?
+U 1 1 5EC46719
+P 2100 6150
+F 0 "#PWR?" H 2100 5900 50  0001 C CNN
+F 1 "GND" H 2105 5977 50  0000 C CNN
+F 2 "" H 2100 6150 50  0001 C CNN
+F 3 "" H 2100 6150 50  0001 C CNN
+	1    2100 6150
+	1    0    0    -1
+$EndComp
+Wire Wire Line
+	2100 5800 2100 6150
+Connection ~ 2100 5800
 $EndSCHEMATC

Commit message: Redraw pcb
Connections:
- net at U1.4 (2Y): now also U3.2 (I2)
- net at U1.6 (3Y): now also U3.1 (I3)
- net at U2.4 (2Y): now also U3.4 (I0)
- net at U2.6 (3Y): now also U3.3 (I1)
Changed lines of the file:
@@
 Sheet 1 2
 Title "Analog inputs 24V"
-Date "2020-02-29"
+Date "2020-03-27"
 Rev "1"
 Comp ""
-Comment1 ""
+Comment1 "SomeController"
 Comment2 "Ivan Semenkov"
 Comment3 ""
@@
 Connection ~ 2900 5800
 Wire Wire Line
-	2850 3600 3650 3600
-Wire Wire Line
-	3650 3600 3650 3500
-Wire Wire Line
-	3650 3500 4000 3500
-Wire Wire Line
-	2850 3500 3550 3500
-Wire Wire Line
-	3550 3500 3550 3400
-Wire Wire Line
-	3550 3400 4000 3400
-Wire Wire Line
-	2850 5500 3850 5500
-Wire Wire Line
-	3850 5500 3850 3300
-Wire Wire Line
-	3850 3300 4000 3300
-Wire Wire Line
-	2850 5400 3750 5400
-Wire Wire Line
-	3750 5400 3750 3200
-Wire Wire Line
-	3750 3200 4000 3200
+	2850 3600 3350 3600
+Wire Wire Line
+	3350 3600 3350 3500
+Wire Wire Line
+	3350 3500 4000 3500
+Wire Wire Line
+	2850 3500 3250 3500
+Wire Wire Line
+	3250 3500 3250 3400
+Wire Wire Line
+	3250 3400 4000 3400
+Wire Wire Line
+	2850 5500 3750 5500
+Wire Wire Line
+	3750 5500 3750 3300
+Wire Wire Line
+	3750 3300 4000 3300
+Wire Wire Line
+	2850 5400 3650 5400
+Wire Wire Line
+	3650 5400 3650 3200
+Wire Wire Line
+	3650 3200 4000 3200
 Wire Notes Line
 	5600 2650 5600 3150
@@
 	2950 4650 3700 4650
 $Comp
-L power:GND #PWR?
+L power:GND #PWR0104
 U 1 1 5EC44226
 P 2900 6150
-F 0 "#PWR?" H 2900 5900 50  0001 C CNN
+F 0 "#PWR0104" H 2900 5900 50  0001 C CNN
 F 1 "GND" H 2905 5977 50  0000 C CNN
 F 2 "" H 2900 6150 50  0001 C CNN
@@
 	2900 5900 2900 6150
 $Comp
-L power:GND #PWR?
+L power:GND #PWR0105
 U 1 1 5EC46719
 P 2100 6150
-F 0 "#PWR?" H 2100 5900 50  0001 C CNN
+F 0 "#PWR0105" H 2100 5900 50  0001 C CNN
 F 1 "GND" H 2105 5977 50  0000 C CNN
 F 2 "" H 2100 6150 50  0001 C CNN
@@
 	2100 5800 2100 6150
 Connection ~ 2100 5800
+Wire Wire Line
+	2850 3700 3450 3700
+Wire Wire Line
+	3450 3700 3450 3600
+Wire Wire Line
+	3450 3600 4000 3600
+Wire Wire Line
+	2850 3800 3550 3800
+Wire Wire Line
+	3550 3800 3550 3700
+Wire Wire Line
+	3550 3700 4000 3700
+Wire Wire Line
+	2850 5600 3850 5600
+Wire Wire Line
+	3850 5600 3850 3800
+Wire Wire Line
+	3850 3800 4000 3800
+Wire Wire Line
+	2850 5700 3950 5700
+Wire Wire Line
+	3950 5700 3950 3900
+Wire Wire Line
+	3950 3900 4000 3900
 $EndSCHEMATC

Commit message: Update Inputs pcb
Parts:
- D1, D2: footprint Diode_THT:D_A-405_P2.54mm_Vertical_AnodeUp -> LED_THT:LED_D3.0mm
- J1, J2: footprint Connector_PinHeader_2.54mm:PinHeader_1x02_P2.54mm_Horizontal -> Connector_PinHeader_2.54mm:PinHeader_1x02_P2.54mm_Vertical
- J3: footprint Connector_PinHeader_2.54mm:PinHeader_1x06_P2.54mm_Horizontal -> Connector_PinHeader_2.54mm:PinHeader_1x06_P2.54mm_Vertical
Changed lines of the file:
@@
 EESchema Schematic File Version 4
-EELAYER 30 0
+LIBS:Inputs_analog_24V_8pcs-cache
+EELAYER 26 0
 EELAYER END
 $Descr A4 11693 8268
@@
 F 0 "J1" H 968 1317 50  0000 C CNN
 F 1 "Screw_Terminal_01x02" H 968 1676 50  0001 C CNN
-F 2 "Connector_PinHeader_2.54mm:PinHeader_1x02_P2.54mm_Horizontal" H 1050 1550 50  0001 C CNN
+F 2 "Connector_PinHeader_2.54mm:PinHeader_1x02_P2.54mm_Vertical" H 1050 1550 50  0001 C CNN
 F 3 "~" H 1050 1550 50  0001 C CNN
 	1    1050 1550
@@
 F 0 "J3" H 5230 3492 50  0000 L CNN
 F 1 "Screw_Terminal_01x06" H 5230 3401 50  0001 L CNN
-F 2 "Connector_PinHeader_2.54mm:PinHeader_1x06_P2.54mm_Horizontal" H 5150 3500 50  0001 C CNN
+F 2 "Connector_PinHeader_2.54mm:PinHeader_1x06_P2.54mm_Vertical" H 5150 3500 50  0001 C CNN
 F 3 "~" H 5150 3500 50  0001 C CNN
 	1    5150 3500
@@
 F 0 "D1" V 1589 2178 50  0000 L CNN
 F 1 "LED" V 1498 2178 50  0000 L CNN
-F 2 "Diode_THT:D_A-405_P2.54mm_Vertical_AnodeUp" H 1550 2100 50  0001 C CNN
+F 2 "LED_THT:LED_D3.0mm" H 1550 2100 50  0001 C CNN
 F 3 "~" H 1550 2100 50  0001 C CNN
 	1    1550 2100
@@
 F 0 "J2" H 2468 1317 50  0000 C CNN
 F 1 "Screw_Terminal_01x02" H 2468 1676 50  0001 C CNN
-F 2 "Connector_PinHeader_2.54mm:PinHeader_1x02_P2.54mm_Horizontal" H 2550 1550 50  0001 C CNN
+F 2 "Connector_PinHeader_2.54mm:PinHeader_1x02_P2.54mm_Vertical" H 2550 1550 50  0001 C CNN
 F 3 "~" H 2550 1550 50  0001 C CNN
 	1    2550 1550
@@
 F 0 "D2" V 3089 2178 50  0000 L CNN
 F 1 "LED" V 2998 2178 50  0000 L CNN
-F 2 "Diode_THT:D_A-405_P2.54mm_Vertical_AnodeUp" H 3050 2100 50  0001 C CNN
+F 2 "LED_THT:LED_D3.0mm" H 3050 2100 50  0001 C CNN
 F 3 "~" H 3050 2100 50  0001 C CNN
 	1    3050 2100

Commit message: Change footprints for ternimals
Parts:
- J1, J2: footprint Connector_PinHeader_2.54mm:PinHeader_1x02_P2.54mm_Vertical -> TerminalBlock_MetzConnect:TerminalBlock_MetzConnect_Type011_RT05502HBWC_1x02_P5.00mm_Horizontal
Changed lines of the file:
@@
 EESchema Schematic File Version 4
-LIBS:Inputs_analog_24V_8pcs-cache
-EELAYER 26 0
+EELAYER 30 0
 EELAYER END
 $Descr A4 11693 8268
@@
 F 0 "J1" H 968 1317 50  0000 C CNN
 F 1 "Screw_Terminal_01x02" H 968 1676 50  0001 C CNN
-F 2 "Connector_PinHeader_2.54mm:PinHeader_1x02_P2.54mm_Vertical" H 1050 1550 50  0001 C CNN
+F 2 "TerminalBlock_MetzConnect:TerminalBlock_MetzConnect_Type011_RT05502HBWC_1x02_P5.00mm_Horizontal" H 1050 1550 50  0001 C CNN
 F 3 "~" H 1050 1550 50  0001 C CNN
 	1    1050 1550
@@
 F 0 "J2" H 2468 1317 50  0000 C CNN
 F 1 "Screw_Terminal_01x02" H 2468 1676 50  0001 C CNN
-F 2 "Connector_PinHeader_2.54mm:PinHeader_1x02_P2.54mm_Vertical" H 2550 1550 50  0001 C CNN
+F 2 "TerminalBlock_MetzConnect:TerminalBlock_MetzConnect_Type011_RT05502HBWC_1x02_P5.00mm_Horizontal" H 2550 1550 50  0001 C CNN
 F 3 "~" H 2550 1550 50  0001 C CNN
 	1    2550 1550
