File: Inputs_analog_24V_8pcs_SMD/Inputs_analog_24V_8pcs.sch (KiCad schematic (older format))
At the start: 27 parts, among them J1 Screw_Terminal_01x02, J2 Screw_Terminal_01x02, J3 Screw_Terminal_01x06, U1 SN74LVC1G14DBVR, U12 SN74LVC1G14DBVR, U13 SN74LVC1G14DBVR, U14 SN74LVC1G14DBVR, U15 SN74LVC1G14DBVR, U16 SN74LVC1G14DBVR, U17 SN74LVC1G14DBVR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

Commit message: Change footprints for ternimals
Parts:
- gave numbers to parts that had none: 1
Changed lines of the file:
@@
 	6750 3550 6800 3550
 $Comp
-L Device:R R?
+L Device:R R52
 U 1 1 5EB619BE
 P 3350 2150
-F 0 "R?" H 3280 2104 50  0000 R CNN
+F 0 "R52" H 3280 2104 50  0000 R CNN
 F 1 "18R" H 3280 2195 50  0000 R CNN
 F 2 "Resistor_SMD:R_0805_2012Metric_Pad1.15x1.40mm_HandSolder" V 3280 2150 50  0001 C CNN
